File: V2/PCB/McPiFace-Pi-4-Audio-V2.0.sch (EAGLE design)
At the start: 11 parts

Commit message: Fixed date/version numbers.
Other:
- note added: "V2.0"
- note removed: "V1.0"
Changed lines of the file:
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@@
 <sheet>
 <plain>
-<text x="238.76" y="7.62" size="2.54" layer="97">V1.0</text>
+<text x="238.76" y="7.62" size="2.54" layer="97">V2.0</text>
 <text x="172.72" y="10.16" size="2.54" layer="97">Stephen Harrison</text>
 <wire x1="0" y1="66.04" x2="76.2" y2="66.04" width="0.1524" layer="97"/>
